File: Documentation/Schematics/Smart_Lamp/Smart_Lamp_v0.1.brd (EAGLE design)
At the start: 60.6 x 47 mm, 18 parts, among them IC1 DS3231/SO, U1 HM-10

Commit message: Small changes to schematic
Parts:
- R7: value 470 -> 1K
Connections:
- net 3.3V: now also C5.1; no longer C5.2
- net N$2: now also C5.2; no longer C5.1
- net S_IN: now also MCU1.11
- net S_OUT: now also MCU1.10
Changed lines of the file:
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@@
 <element name="R4" library="rcl" package="0207/10" value="10K" x="52.07" y="36.83"/>
 <element name="R5" library="microbuilder" package="0805-NO" value="10K" x="24.13" y="41.91"/>
-<element name="R7" library="rcl" package="0207/10" value="470" x="39.37" y="36.83"/>
+<element name="R7" library="rcl" package="0207/10" value="1K" x="39.37" y="36.83"/>
 <element name="R8" library="rcl" package="0207/10" value="470" x="26.67" y="36.83"/>
 <element name="U1" library="HM-10_BLE" package="HM-10" value="HM-10" x="8.89" y="15.24" rot="R180"/>
@@
 <contactref element="IC1" pad="2"/>
 <contactref element="R7" pad="1"/>
-<contactref element="C5" pad="2"/>
 <contactref element="C3" pad="1"/>
+<contactref element="C5" pad="1"/>
 <wire x1="46.99" y1="36.83" x2="44.13" y2="41.91" width="0" layer="19" extent="1-1"/>
 <wire x1="45.72" y1="30.48" x2="46.99" y2="36.83" width="0" layer="19" extent="1-1"/>
@@
 <wire x1="29.53" y1="41.91" x2="35.88" y2="41.91" width="0" layer="19" extent="1-1"/>
 <wire x1="23.18" y1="41.91" x2="29.53" y2="41.91" width="0" layer="19" extent="1-1"/>
-<wire x1="33.02" y1="29.21" x2="34.29" y2="36.83" width="0" layer="19" extent="1-1"/>
-<wire x1="36.83" y1="29.21" x2="33.02" y2="29.21" width="0" layer="19" extent="1-1"/>
-<wire x1="23.28" y1="27.94" x2="33.02" y2="29.21" width="0" layer="19" extent="1-1"/>
+<wire x1="36.83" y1="29.21" x2="34.29" y2="36.83" width="0" layer="19" extent="1-1"/>
+<wire x1="30.48" y1="29.21" x2="36.83" y2="29.21" width="0" layer="19" extent="1-1"/>
+<wire x1="23.28" y1="27.94" x2="30.48" y2="29.21" width="0" layer="19" extent="1-1"/>
 <wire x1="20.32" y1="15.24" x2="23.28" y2="27.94" width="0" layer="19" extent="1-1"/>
 <wire x1="29.21" y1="6.5278" x2="20.32" y2="15.24" width="0" layer="19" extent="1-1"/>
@@
 <signal name="S_OUT">
 <contactref element="U1" pad="1"/>
+<contactref element="MCU1" pad="10"/>
+<wire x1="15.66" y1="8.89" x2="30.48" y2="22.86" width="0" layer="19" extent="1-1"/>
 </signal>
 <signal name="S_IN">
 <contactref element="U1" pad="2"/>
+<contactref element="MCU1" pad="11"/>
+<wire x1="15.66" y1="10.39" x2="27.94" y2="22.86" width="0" layer="19" extent="1-1"/>
 </signal>
 <signal name="N$9">
@@
 </signal>
 <signal name="N$2">
+<contactref element="C5" pad="2"/>
 <contactref element="S1" pad="S"/>
-<contactref element="C5" pad="1"/>
-<wire x1="43.18" y1="7.62" x2="30.48" y2="29.21" width="0" layer="19" extent="1-1"/>
+<wire x1="43.18" y1="7.62" x2="33.02" y2="29.21" width="0" layer="19" extent="1-1"/>
 </signal>
 </signals>
