File: Documentation/Schematics/SmartLamp/SmartLamp.brd (EAGLE design)
At the start: 78.4 x 49.5 mm, 25 parts, among them J1 POWER_JACKPTH_BREAD, Q1 IRF1404, Q2 IRF1404, Q3 IRF1404, U1 HM-10, U2 DS3231MZ

Commit message: Added datasheet for new mosfet IRLZ44n, small changes to HM-10 test program.
Parts:
- Q1, Q2, Q3: value IRF1404 -> IRLZ44Z
- moved Q2 11.4 mm to (48.3, 33.0)
- moved Q3 11.4 mm to (36.8, 33.0)
Changed lines of the file:
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@@
 <element name="R8" library="rcl" package="0309/12" value="470" x="31.75" y="19.05"/>
 <element name="U1" library="HM-10_BLE" package="HM-10" value="HM-10" x="15.24" y="40.64" rot="R90"/>
-<element name="Q1" library="transistor-power" package="TO220BH" value="IRF1404" x="59.69" y="33.02"/>
-<element name="Q2" library="transistor-power" package="TO220BH" value="IRF1404" x="36.83" y="33.02"/>
-<element name="Q3" library="transistor-power" package="TO220BH" value="IRF1404" x="48.26" y="33.02"/>
 <element name="LED_STRIP" library="pinhead" package="1X04" value="" x="73.66" y="30.48" rot="R90"/>
 <element name="R3" library="rcl" package="0207/10" value="220" x="45.72" y="17.78" rot="R90"/>
@@
 <attribute name="MANUFACTURER_PART_NUMBER" value="DS3231MZ" x="17.78" y="29.21" size="1.778" layer="27" display="off"/>
 </element>
+<element name="Q1" library="transistor-power" package="TO220BH" value="IRLZ44Z" x="59.69" y="33.02"/>
+<element name="Q2" library="transistor-power" package="TO220BH" value="IRLZ44Z" x="48.26" y="33.02"/>
+<element name="Q3" library="transistor-power" package="TO220BH" value="IRLZ44Z" x="36.83" y="33.02"/>
 </elements>
 <signals>
@@
 <contactref element="U1" pad="22"/>
 <contactref element="LED1" pad="K"/>
-<contactref element="Q1" pad="S"/>
-<contactref element="Q2" pad="S"/>
-<contactref element="Q3" pad="S"/>
 <contactref element="J1" pad="GND"/>
 <contactref element="C1" pad="2"/>
@@
 <contactref element="G1" pad="-"/>
 <contactref element="U2" pad="5"/>
+<contactref element="Q1" pad="S"/>
+<contactref element="Q2" pad="S"/>
+<contactref element="Q3" pad="S"/>
 <wire x1="67.31" y1="29.21" x2="73.38" y2="43.18" width="0" layer="19" extent="1-1"/>
-<wire x1="62.23" y1="26.67" x2="67.31" y2="29.21" width="0" layer="19" extent="1-1"/>
-<wire x1="50.8" y1="26.67" x2="62.23" y2="26.67" width="0" layer="19" extent="1-1"/>
-<wire x1="39.37" y1="26.67" x2="50.8" y2="26.67" width="0" layer="19" extent="1-1"/>
-<wire x1="28.96" y1="35.41" x2="39.37" y2="26.67" width="0" layer="19" extent="1-1"/>
-<wire x1="26.89" y1="33.87" x2="28.96" y2="35.41" width="0" layer="19" extent="1-1"/>
-<wire x1="20.2438" y1="27.305" x2="26.89" y2="33.87" width="0" layer="19" extent="1-1"/>
-<wire x1="20.32" y1="21.59" x2="20.2438" y2="27.305" width="0" layer="19" extent="1-1"/>
-<wire x1="15.24" y1="21.59" x2="20.32" y2="21.59" width="0" layer="19" extent="1-1"/>
+<wire x1="72.04" y1="12.7" x2="67.31" y2="29.21" width="0" layer="19" extent="1-1"/>
+<wire x1="44.45" y1="2.7178" x2="72.04" y2="12.7" width="0" layer="19" extent="1-1"/>
+<wire x1="33.02" y1="6.35" x2="44.45" y2="2.7178" width="0" layer="19" extent="1-1"/>
+<wire x1="30.48" y1="6.35" x2="33.02" y2="6.35" width="0" layer="19" extent="1-1"/>
+<wire x1="13.97" y1="5.08" x2="30.48" y2="6.35" width="0" layer="19" extent="1-1"/>
+<wire x1="5.08" y1="2.54" x2="13.97" y2="5.08" width="0" layer="19" extent="1-1"/>
+<wire x1="15.24" y1="21.59" x2="13.97" y2="5.08" width="0" layer="19" extent="1-1"/>
+<wire x1="20.32" y1="21.59" x2="15.24" y2="21.59" width="0" layer="19" extent="1-1"/>
+<wire x1="20.2438" y1="27.305" x2="20.32" y2="21.59" width="0" layer="19" extent="1-1"/>
+<wire x1="26.89" y1="33.87" x2="20.2438" y2="27.305" width="0" layer="19" extent="1-1"/>
+<wire x1="28.96" y1="35.41" x2="26.89" y2="33.87" width="0" layer="19" extent="1-1"/>
 <wire x1="11.43" y1="30.48" x2="20.2438" y2="27.305" width="0" layer="19" extent="1-1"/>
 <wire x1="28.96" y1="45.91" x2="28.96" y2="35.41" width="0" layer="19" extent="1-1"/>
 <wire x1="26.89" y1="47.41" x2="28.96" y2="45.91" width="0" layer="19" extent="1-1"/>
-<wire x1="13.97" y1="5.08" x2="15.24" y2="21.59" width="0" layer="19" extent="1-1"/>
-<wire x1="5.08" y1="2.54" x2="13.97" y2="5.08" width="0" layer="19" extent="1-1"/>
-<wire x1="30.48" y1="6.35" x2="13.97" y2="5.08" width="0" layer="19" extent="1-1"/>
-<wire x1="33.02" y1="6.35" x2="30.48" y2="6.35" width="0" layer="19" extent="1-1"/>
-<wire x1="44.45" y1="2.7178" x2="33.02" y2="6.35" width="0" layer="19" extent="1-1"/>
-<wire x1="72.04" y1="12.7" x2="62.23" y2="26.67" width="0" layer="19" extent="1-1"/>
+<wire x1="62.23" y1="26.67" x2="5.08" y2="2.54" width="0" layer="19" extent="1-1"/>
+<wire x1="50.8" y1="26.67" x2="62.23" y2="26.67" width="0" layer="19" extent="1-1"/>
+<wire x1="39.37" y1="26.67" x2="50.8" y2="26.67" width="0" layer="19" extent="1-1"/>
 </signal>
 <signal name="SDA">
@@
 </signal>
 <signal name="N$3" class="1">
+<contactref element="LED_STRIP" pad="2"/>
 <contactref element="Q1" pad="D"/>
-<contactref element="LED_STRIP" pad="2"/>
 <wire x1="59.69" y1="26.67" x2="73.66" y2="29.21" width="0" layer="19" extent="1-1"/>
 </signal>
 <signal name="N$4" class="1">
+<contactref element="LED_STRIP" pad="3"/>
 <contactref element="Q2" pad="D"/>
-<contactref element="LED_STRIP" pad="3"/>
-<wire x1="36.83" y1="26.67" x2="73.66" y2="31.75" width="0" layer="19" extent="1-1"/>
+<wire x1="48.26" y1="26.67" x2="73.66" y2="31.75" width="0" layer="19" extent="1-1"/>
 </signal>
 <signal name="N$6" class="1">
+<contactref element="LED_STRIP" pad="4"/>
 <contactref element="Q3" pad="D"/>
-<contactref element="LED_STRIP" pad="4"/>
-<wire x1="48.26" y1="26.67" x2="73.66" y2="34.29" width="0" layer="19" extent="1-1"/>
+<wire x1="36.83" y1="26.67" x2="73.66" y2="34.29" width="0" layer="19" extent="1-1"/>
 </signal>
 <signal name="N$7">
+<contactref element="R3" pad="2"/>
 <contactref element="Q1" pad="G"/>
-<contactref element="R3" pad="2"/>
-<wire x1="45.72" y1="22.86" x2="57.15" y2="26.67" width="0" layer="19" extent="1-1"/>
+<wire x1="57.15" y1="26.67" x2="45.72" y2="22.86" width="0" layer="19" extent="1-1"/>
 </signal>
 <signal name="N$8">
 <contactref element="R4" pad="2"/>
 <contactref element="Q2" pad="G"/>
-<wire x1="34.29" y1="26.67" x2="40.64" y2="22.86" width="0" layer="19" extent="1-1"/>
+<wire x1="45.72" y1="26.67" x2="40.64" y2="22.86" width="0" layer="19" extent="1-1"/>
 </signal>
 <signal name="N$11">
 <contactref element="R5" pad="2"/>
 <contactref element="Q3" pad="G"/>
-<wire x1="45.72" y1="26.67" x2="48.26" y2="22.86" width="0" layer="19" extent="1-1"/>
+<wire x1="34.29" y1="26.67" x2="48.26" y2="22.86" width="0" layer="19" extent="1-1"/>
 </signal>
 <signal name="RED">

Commit message: Changed dip switch to cut GND instead of VCC to bluetooth module.
Connections:
- net +3V3: now also C4.1; no longer S1.1
- net GND: now also S1.4; no longer U1.13
- net N$1: no longer C4.2
- net N$2: now also S1.1, U1.13; no longer C4.1, S1.4
Changed lines of the file:
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@@
 <signal name="GND">
 <contactref element="LF33ABV" pad="2"/>
-<contactref element="U1" pad="13"/>
 <contactref element="U1" pad="14"/>
 <contactref element="U1" pad="21"/>
@@
 <contactref element="Q2" pad="S"/>
 <contactref element="Q3" pad="S"/>
+<contactref element="S1" pad="4"/>
 <wire x1="67.31" y1="29.21" x2="73.38" y2="43.18" width="0" layer="19" extent="1-1"/>
-<wire x1="72.04" y1="12.7" x2="67.31" y2="29.21" width="0" layer="19" extent="1-1"/>
-<wire x1="44.45" y1="2.7178" x2="72.04" y2="12.7" width="0" layer="19" extent="1-1"/>
-<wire x1="33.02" y1="6.35" x2="44.45" y2="2.7178" width="0" layer="19" extent="1-1"/>
-<wire x1="30.48" y1="6.35" x2="33.02" y2="6.35" width="0" layer="19" extent="1-1"/>
-<wire x1="13.97" y1="5.08" x2="30.48" y2="6.35" width="0" layer="19" extent="1-1"/>
-<wire x1="5.08" y1="2.54" x2="13.97" y2="5.08" width="0" layer="19" extent="1-1"/>
-<wire x1="15.24" y1="21.59" x2="13.97" y2="5.08" width="0" layer="19" extent="1-1"/>
-<wire x1="20.32" y1="21.59" x2="15.24" y2="21.59" width="0" layer="19" extent="1-1"/>
-<wire x1="20.2438" y1="27.305" x2="20.32" y2="21.59" width="0" layer="19" extent="1-1"/>
-<wire x1="26.89" y1="33.87" x2="20.2438" y2="27.305" width="0" layer="19" extent="1-1"/>
-<wire x1="28.96" y1="35.41" x2="26.89" y2="33.87" width="0" layer="19" extent="1-1"/>
-<wire x1="11.43" y1="30.48" x2="20.2438" y2="27.305" width="0" layer="19" extent="1-1"/>
+<wire x1="62.23" y1="26.67" x2="67.31" y2="29.21" width="0" layer="19" extent="1-1"/>
+<wire x1="50.8" y1="26.67" x2="62.23" y2="26.67" width="0" layer="19" extent="1-1"/>
+<wire x1="39.37" y1="26.67" x2="50.8" y2="26.67" width="0" layer="19" extent="1-1"/>
+<wire x1="28.96" y1="35.41" x2="39.37" y2="26.67" width="0" layer="19" extent="1-1"/>
 <wire x1="28.96" y1="45.91" x2="28.96" y2="35.41" width="0" layer="19" extent="1-1"/>
 <wire x1="26.89" y1="47.41" x2="28.96" y2="45.91" width="0" layer="19" extent="1-1"/>
-<wire x1="62.23" y1="26.67" x2="5.08" y2="2.54" width="0" layer="19" extent="1-1"/>
-<wire x1="50.8" y1="26.67" x2="62.23" y2="26.67" width="0" layer="19" extent="1-1"/>
-<wire x1="39.37" y1="26.67" x2="50.8" y2="26.67" width="0" layer="19" extent="1-1"/>
+<wire x1="20.2438" y1="27.305" x2="28.96" y2="35.41" width="0" layer="19" extent="1-1"/>
+<wire x1="20.32" y1="21.59" x2="20.2438" y2="27.305" width="0" layer="19" extent="1-1"/>
+<wire x1="15.24" y1="21.59" x2="20.32" y2="21.59" width="0" layer="19" extent="1-1"/>
+<wire x1="11.43" y1="30.48" x2="20.2438" y2="27.305" width="0" layer="19" extent="1-1"/>
+<wire x1="13.97" y1="5.08" x2="15.24" y2="21.59" width="0" layer="19" extent="1-1"/>
+<wire x1="7.62" y1="2.54" x2="13.97" y2="5.08" width="0" layer="19" extent="1-1"/>
+<wire x1="5.08" y1="2.54" x2="7.62" y2="2.54" width="0" layer="19" extent="1-1"/>
+<wire x1="30.48" y1="6.35" x2="13.97" y2="5.08" width="0" layer="19" extent="1-1"/>
+<wire x1="33.02" y1="6.35" x2="30.48" y2="6.35" width="0" layer="19" extent="1-1"/>
+<wire x1="44.45" y1="2.7178" x2="33.02" y2="6.35" width="0" layer="19" extent="1-1"/>
+<wire x1="72.04" y1="12.7" x2="62.23" y2="26.67" width="0" layer="19" extent="1-1"/>
 </signal>
 <signal name="SDA">
@@
 <contactref element="R3" pad="2"/>
 <contactref element="Q1" pad="G"/>
-<wire x1="57.15" y1="26.67" x2="45.72" y2="22.86" width="0" layer="19" extent="1-1"/>
+<wire x1="45.72" y1="22.86" x2="57.15" y2="26.67" width="0" layer="19" extent="1-1"/>
 </signal>
 <signal name="N$8">
 <contactref element="R4" pad="2"/>
 <contactref element="Q2" pad="G"/>
-<wire x1="45.72" y1="26.67" x2="40.64" y2="22.86" width="0" layer="19" extent="1-1"/>
+<wire x1="40.64" y1="22.86" x2="45.72" y2="26.67" width="0" layer="19" extent="1-1"/>
 </signal>
 <signal name="N$11">
@@
 <signal name="N$1">
 <contactref element="U1" pad="12"/>
-<contactref element="C4" pad="2"/>
-<wire x1="25.39" y1="33.87" x2="29.21" y2="30.48" width="0" layer="19" extent="1-1"/>
-</signal>
-<signal name="N$2">
-<contactref element="S1" pad="4"/>
-<contactref element="C4" pad="1"/>
-<wire x1="7.62" y1="2.54" x2="29.21" y2="27.94" width="0" layer="19" extent="1-1"/>
 </signal>
 <signal name="+3V3" class="2">
@@
 <contactref element="LF33ABV" pad="3"/>
 <contactref element="R7" pad="1"/>
-<contactref element="S1" pad="1"/>
 <contactref element="C3" pad="1"/>
 <contactref element="U2" pad="2"/>
+<contactref element="C4" pad="1"/>
 <wire x1="43.18" y1="12.7" x2="67.31" y2="26.67" width="0" layer="19" extent="1-1"/>
 <wire x1="38.1" y1="11.43" x2="43.18" y2="12.7" width="0" layer="19" extent="1-1"/>
 <wire x1="38.1381" y1="15.3416" x2="38.1" y2="11.43" width="0" layer="19" extent="1-1"/>
 <wire x1="38.1" y1="22.86" x2="38.1381" y2="15.3416" width="0" layer="19" extent="1-1"/>
+<wire x1="29.21" y1="27.94" x2="38.1" y2="22.86" width="0" layer="19" extent="1-1"/>
+<wire x1="20.32" y1="24.13" x2="29.21" y2="27.94" width="0" layer="19" extent="1-1"/>
+<wire x1="15.3162" y1="29.845" x2="20.32" y2="24.13" width="0" layer="19" extent="1-1"/>
 <wire x1="46.99" y1="2.7178" x2="43.18" y2="12.7" width="0" layer="19" extent="1-1"/>
-<wire x1="20.32" y1="24.13" x2="38.1" y2="22.86" width="0" layer="19" extent="1-1"/>
-<wire x1="15.3162" y1="29.845" x2="20.32" y2="24.13" width="0" layer="19" extent="1-1"/>
-<wire x1="7.62" y1="10.16" x2="20.32" y2="24.13" width="0" layer="19" extent="1-1"/>
+</signal>
+<signal name="N$2">
+<contactref element="U1" pad="13"/>
+<contactref element="S1" pad="1"/>
+<wire x1="7.62" y1="10.16" x2="26.89" y2="33.87" width="0" layer="19" extent="1-1"/>
 </signal>
 </signals>

Commit message: Fixed IO connections to micro, in schematic and main.cpp
Connections:
- removed net N$9: R8.2, U1.24
- new net BLU_STATE: MCU1.3, R8.2, U1.24
- net !BLU_RES: now also MCU1.12; no longer MCU1.5
- net !INT_SQW: now also MCU1.13; no longer MCU1.9
- net GR: now also MCU1.11; no longer MCU1.7
- net RED: now also MCU1.10; no longer MCU1.6
- net SCL: now also MCU1.9; no longer MCU1.13
- net SDA: now also MCU1.7; no longer MCU1.12
- net S_IN: now also MCU1.5, U1.1; no longer MCU1.11, U1.2
- net S_OUT: now also MCU1.6, U1.2; no longer MCU1.10, U1.1
- net S_OUT_DEBUG: now also MCU1.2; no longer MCU1.3
Changed lines of the file:
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@@
 <signal name="SDA">
 <contactref element="R1" pad="2"/>
-<contactref element="MCU1" pad="12"/>
 <contactref element="U2" pad="7"/>
-<wire x1="11.43" y1="25.4" x2="20.2438" y2="29.845" width="0" layer="19" extent="1-1"/>
+<contactref element="MCU1" pad="7"/>
 <wire x1="25.4381" y1="15.3416" x2="20.2438" y2="29.845" width="0" layer="19" extent="1-1"/>
+<wire x1="3.81" y1="15.24" x2="25.4381" y2="15.3416" width="0" layer="19" extent="1-1"/>
 </signal>
 <signal name="SCL">
 <contactref element="R2" pad="2"/>
-<contactref element="MCU1" pad="13"/>
 <contactref element="U2" pad="8"/>
-<wire x1="11.43" y1="27.94" x2="20.2438" y2="31.115" width="0" layer="19" extent="1-1"/>
-<wire x1="25.4" y1="11.43" x2="20.2438" y2="31.115" width="0" layer="19" extent="1-1"/>
+<contactref element="MCU1" pad="9"/>
+<wire x1="11.43" y1="17.78" x2="20.2438" y2="31.115" width="0" layer="19" extent="1-1"/>
+<wire x1="25.4" y1="11.43" x2="11.43" y2="17.78" width="0" layer="19" extent="1-1"/>
 </signal>
 <signal name="3V3" class="2">
@@
 </signal>
 <signal name="!INT_SQW">
-<contactref element="MCU1" pad="9"/>
 <contactref element="IDC1" pad="7"/>
 <contactref element="U2" pad="3"/>
-<wire x1="11.43" y1="17.78" x2="15.3162" y2="28.575" width="0" layer="19" extent="1-1"/>
-<wire x1="30.48" y1="3.81" x2="11.43" y2="17.78" width="0" layer="19" extent="1-1"/>
+<contactref element="MCU1" pad="13"/>
+<wire x1="11.43" y1="27.94" x2="15.3162" y2="28.575" width="0" layer="19" extent="1-1"/>
+<wire x1="30.48" y1="3.81" x2="15.3162" y2="28.575" width="0" layer="19" extent="1-1"/>
 </signal>
 <signal name="RESET">
@@
 </signal>
 <signal name="S_OUT">
-<contactref element="U1" pad="1"/>
-<contactref element="MCU1" pad="10"/>
-<wire x1="11.43" y1="20.32" x2="8.89" y2="33.87" width="0" layer="19" extent="1-1"/>
+<contactref element="MCU1" pad="6"/>
+<contactref element="U1" pad="2"/>
+<wire x1="3.81" y1="17.78" x2="10.39" y2="33.87" width="0" layer="19" extent="1-1"/>
 </signal>
 <signal name="S_IN">
-<contactref element="U1" pad="2"/>
-<contactref element="MCU1" pad="11"/>
-<wire x1="11.43" y1="22.86" x2="10.39" y2="33.87" width="0" layer="19" extent="1-1"/>
+<contactref element="MCU1" pad="5"/>
+<contactref element="U1" pad="1"/>
+<wire x1="3.81" y1="20.32" x2="8.89" y2="33.87" width="0" layer="19" extent="1-1"/>
 </signal>
-<signal name="N$9">
+<signal name="BLU_STATE">
 <contactref element="U1" pad="24"/>
 <contactref element="R8" pad="2"/>
+<contactref element="MCU1" pad="3"/>
+<wire x1="3.81" y1="25.4" x2="23.89" y2="47.41" width="0" layer="19" extent="1-1"/>
 <wire x1="38.1" y1="19.05" x2="23.89" y2="47.41" width="0" layer="19" extent="1-1"/>
 </signal>
@@
 <signal name="RED">
 <contactref element="R3" pad="1"/>
-<contactref element="MCU1" pad="6"/>
-<wire x1="3.81" y1="17.78" x2="45.72" y2="12.7" width="0" layer="19" extent="1-1"/>
+<contactref element="MCU1" pad="10"/>
+<wire x1="11.43" y1="20.32" x2="45.72" y2="12.7" width="0" layer="19" extent="1-1"/>
 </signal>
 <signal name="GR">
 <contactref element="R4" pad="1"/>
-<contactref element="MCU1" pad="7"/>
 <contactref element="IDC1" pad="1"/>
+<contactref element="MCU1" pad="11"/>
 <wire x1="22.86" y1="3.81" x2="40.64" y2="12.7" width="0" layer="19" extent="1-1"/>
-<wire x1="3.81" y1="15.24" x2="22.86" y2="3.81" width="0" layer="19" extent="1-1"/>
+<wire x1="11.43" y1="22.86" x2="22.86" y2="3.81" width="0" layer="19" extent="1-1"/>
 </signal>
 <signal name="BLUE">
@@
 </signal>
 <signal name="!BLU_RES">
-<contactref element="MCU1" pad="5"/>
 <contactref element="U1" pad="11"/>
-<wire x1="3.81" y1="20.32" x2="23.89" y2="33.87" width="0" layer="19" extent="1-1"/>
+<contactref element="MCU1" pad="12"/>
+<wire x1="11.43" y1="25.4" x2="23.89" y2="33.87" width="0" layer="19" extent="1-1"/>
 </signal>
 <signal name="VBAT">
@@
 </signal>
 <signal name="S_OUT_DEBUG">
-<contactref element="MCU1" pad="3"/>
 <contactref element="IDC1" pad="6"/>
-<wire x1="3.81" y1="25.4" x2="27.94" y2="6.35" width="0" layer="19" extent="1-1"/>
+<contactref element="MCU1" pad="2"/>
+<wire x1="3.81" y1="27.94" x2="27.94" y2="6.35" width="0" layer="19" extent="1-1"/>
 </signal>
 <signal name="N$1">

Commit message: Fixed cap on HM-10 module...
Connections:
- removed net N$1 (its old number): U1.12
- net +3V3: now also U1.12
- net GND: now also C4.2
Changed lines of the file:
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@@
 <contactref element="C2" pad="2"/>
 <contactref element="MCU1" pad="14"/>
-<contactref element="S1" pad="3"/>
 <contactref element="C3" pad="2"/>
 <contactref element="G1" pad="-"/>
@@
 <contactref element="Q2" pad="S"/>
 <contactref element="Q3" pad="S"/>
+<contactref element="C4" pad="2"/>
 <contactref element="S1" pad="4"/>
+<contactref element="S1" pad="3"/>
 <wire x1="67.31" y1="29.21" x2="73.38" y2="43.18" width="0" layer="19" extent="1-1"/>
 <wire x1="62.23" y1="26.67" x2="67.31" y2="29.21" width="0" layer="19" extent="1-1"/>
 <wire x1="50.8" y1="26.67" x2="62.23" y2="26.67" width="0" layer="19" extent="1-1"/>
 <wire x1="39.37" y1="26.67" x2="50.8" y2="26.67" width="0" layer="19" extent="1-1"/>
-<wire x1="28.96" y1="35.41" x2="39.37" y2="26.67" width="0" layer="19" extent="1-1"/>
-<wire x1="28.96" y1="45.91" x2="28.96" y2="35.41" width="0" layer="19" extent="1-1"/>
-<wire x1="26.89" y1="47.41" x2="28.96" y2="45.91" width="0" layer="19" extent="1-1"/>
-<wire x1="20.2438" y1="27.305" x2="28.96" y2="35.41" width="0" layer="19" extent="1-1"/>
+<wire x1="29.21" y1="30.48" x2="39.37" y2="26.67" width="0" layer="19" extent="1-1"/>
+<wire x1="28.96" y1="35.41" x2="29.21" y2="30.48" width="0" layer="19" extent="1-1"/>
+<wire x1="20.2438" y1="27.305" x2="29.21" y2="30.48" width="0" layer="19" extent="1-1"/>
 <wire x1="20.32" y1="21.59" x2="20.2438" y2="27.305" width="0" layer="19" extent="1-1"/>
 <wire x1="15.24" y1="21.59" x2="20.32" y2="21.59" width="0" layer="19" extent="1-1"/>
 <wire x1="11.43" y1="30.48" x2="20.2438" y2="27.305" width="0" layer="19" extent="1-1"/>
+<wire x1="28.96" y1="45.91" x2="28.96" y2="35.41" width="0" layer="19" extent="1-1"/>
+<wire x1="26.89" y1="47.41" x2="28.96" y2="45.91" width="0" layer="19" extent="1-1"/>
 <wire x1="13.97" y1="5.08" x2="15.24" y2="21.59" width="0" layer="19" extent="1-1"/>
 <wire x1="7.62" y1="2.54" x2="13.97" y2="5.08" width="0" layer="19" extent="1-1"/>
@@
 <wire x1="3.81" y1="27.94" x2="27.94" y2="6.35" width="0" layer="19" extent="1-1"/>
 </signal>
-<signal name="N$1">
-<contactref element="U1" pad="12"/>
-</signal>
 <signal name="+3V3" class="2">
 <contactref element="R6" pad="1"/>
@@
 <contactref element="U2" pad="2"/>
 <contactref element="C4" pad="1"/>
+<contactref element="U1" pad="12"/>
 <wire x1="43.18" y1="12.7" x2="67.31" y2="26.67" width="0" layer="19" extent="1-1"/>
 <wire x1="38.1" y1="11.43" x2="43.18" y2="12.7" width="0" layer="19" extent="1-1"/>
@@
 <wire x1="38.1" y1="22.86" x2="38.1381" y2="15.3416" width="0" layer="19" extent="1-1"/>
 <wire x1="29.21" y1="27.94" x2="38.1" y2="22.86" width="0" layer="19" extent="1-1"/>
+<wire x1="25.39" y1="33.87" x2="29.21" y2="27.94" width="0" layer="19" extent="1-1"/>
 <wire x1="20.32" y1="24.13" x2="29.21" y2="27.94" width="0" layer="19" extent="1-1"/>
 <wire x1="15.3162" y1="29.845" x2="20.32" y2="24.13" width="0" layer="19" extent="1-1"/>
 <wire x1="46.99" y1="2.7178" x2="43.18" y2="12.7" width="0" layer="19" extent="1-1"/>
 </signal>
-<signal name="N$2">
+<signal name="N$1">
+<contactref element="S1" pad="1"/>
 <contactref element="U1" pad="13"/>
-<contactref element="S1" pad="1"/>
 <wire x1="7.62" y1="10.16" x2="26.89" y2="33.87" width="0" layer="19" extent="1-1"/>
 </signal>
